File: Hardware/Lora/rns-gate.kicad_pcb (KiCad board)
At the start: 2 copper layers, 48 x 46 mm, 6 parts, among them J2 Conn_02x13_Odd_Even, U1 E22-900M30S-SX1262

Commit message: Update Lora module
Parts:
- added C1: C_Polarized_Small, Capacitor_Tantalum_SMD:CP_EIA-7343-43_Kemet-X_Pad2.25x2.55mm_HandSolder, F.Cu at (180.8, 56.3)
- added C2: C_Small, Capacitor_SMD:C_0805_2012Metric_Pad1.18x1.45mm_HandSolder, F.Cu at (171.2, 56.5)
- added C3: C_Small, Capacitor_SMD:C_0805_2012Metric_Pad1.18x1.45mm_HandSolder, F.Cu at (173.7, 56.5)
Routing:
- net +5V: track 36.4 -> 51.9 mm
