File: Hardware/Audio/rns-gate.kicad_pcb (KiCad board)
At the start: 2 copper layers, 48 x 46 mm, 17 parts, among them J1 Conn_01x13, J2 Conn_02x13_Odd_Even, J3 Conn_01x02, J5 Conn_01x04, Q1 2N7002

Commit message: Update Audio module
Parts:
- added R3: tune, Resistor_SMD:R_0805_2012Metric, F.Cu at (167.6, 75.8)
- added R4: tune, Resistor_SMD:R_0805_2012Metric, F.Cu at (167.6, 71.3)
- added R5: tune, Resistor_SMD:R_0805_2012Metric, F.Cu at (167.6, 63.9)
- added R6: tune, Resistor_SMD:R_0805_2012Metric, F.Cu at (167.6, 59.6)
- C1, C2, C3, C4: value C_Small -> 1u
- R1: value R_Small -> 470
- R2: value R_Small -> 10K
- REF1, REF2, REF3, REF4: value MountingHole_2.2mm_M2_Pad_Via -> MountingHole_3.5mm; footprint MountingHole:MountingHole_2.2mm_M2_Pad_Via -> MountingHole:MountingHole_3.5mm
- RV1, RV2: value R_Potentiometer -> 5K
Routing:
- net Net-(RV1-Pad2): track 12.8 -> 23.2 mm, vias 0 -> 1
- net Net-(C2-Pad1): track 4.64 -> 14.3 mm
- net Net-(C4-Pad1): track 4.64 -> 12.1 mm, vias 0 -> 1
- net Net-(RV2-Pad1): track 4.64 -> 11.5 mm
