File: Hardware/Audio/rns-gate.kicad_sch (KiCad schematic)
At the start: 13 parts, among them J1 Conn_01x13, J2 Conn_02x13_Odd_Even, J3 Conn_01x02, J5 Conn_01x04, Q1 2N7002

Commit message: Update Audio module
Parts:
- added R3, R4, R5, R6: tune, Resistor_SMD:R_0805_2012Metric, symbol Device:R_Small
- C3: value C_Small -> 1u
Connections:
- net GND: now also R4.1, R6.1
- net at C1.2, RV2.1: now also R5.2
- net at C2.1, RV2.2: now also R5.1, R6.2
- net at C4.1, RV1.1: now also R3.2
- net at J5.2 (Pin_2), RV1.2: now also R3.1, R4.2
Other:
- moved on the sheet: C1, RV1
